File: pcb/PowerBoard/PowerBoard.sch (KiCad schematic (older format))
At the start: 9 parts, among them P1 Motor battery, P2 CONN_01X06, P3 Arduino battery, SW1 OnOffDoubleSwitch

Commit message: power board ready
Connections:
- net GND: now reaches DCDC1.4 (OUT-), DCDC2.4 (OUT-), DCDC3.4 (OUT-), P2.1 (P1), P2.3 (P3), P2.5 (P5)
Changed lines of the file:
@@
 Connection ~ 5000 1800
 Wire Wire Line
-	5700 2000 5000 2000
+	4700 2000 5700 2000
 Connection ~ 5000 2000
 Wire Wire Line
@@
 Wire Wire Line
 	1750 1350 2350 1350
+$Comp
+L GND #PWR?
+U 1 1 5783E56C
+P 4700 2150
+F 0 "#PWR?" H 4700 1900 50  0001 C CNN
+F 1 "GND" H 4700 2000 50  0000 C CNN
+F 2 "" H 4700 2150 50  0000 C CNN
+F 3 "" H 4700 2150 50  0000 C CNN
+	1    4700 2150
+	1    0    0    -1
+$EndComp
+Wire Wire Line
+	4700 2000 4700 2150
 $EndSCHEMATC
