File: pcb/MainBoard/MainBoard.sch (KiCad schematic (older format))
At the start: 8 parts

Commit message: PCB design finished
Parts:
- removed C_BULK_2, C_BULK_3: 10-100uF, Capacitors_ThroughHole:C_Radial_D6.3_L11.2_P2.5, symbol CP
- removed C_BULK_6, C_BULK_7: 10-100uF, Capacitors_SMD:C_1206_HandSoldering, symbol C
- renumbered C_BULK_1 to C_5VBULK_1, C_BULK_4 to C_5VBULK_2, C_BULK_5 to C_5VBULK_3
Other:
- moved on the sheet: C_5VBULK_2, C_5VBULK_3
Changed lines of the file:
@@
 $EndComp
 $Comp
-L C C_BULK_4
+L C C_5VBULK_2
 U 1 1 57F9FCC5
-P 3500 6250
-F 0 "C_BULK_4" H 3525 6350 50  0000 L CNN
-F 1 "10-100uF" H 3525 6150 50  0000 L CNN
-F 2 "Capacitors_SMD:C_1206_HandSoldering" H 3538 6100 50  0001 C CNN
-F 3 "" H 3500 6250 50  0000 C CNN
-	1    3500 6250
+P 2450 6250
+F 0 "C_5VBULK_2" H 2475 6350 50  0000 L CNN
+F 1 "10-100uF" H 2475 6150 50  0000 L CNN
+F 2 "Capacitors_SMD:C_1206_HandSoldering" H 2488 6100 50  0001 C CNN
+F 3 "" H 2450 6250 50  0000 C CNN
+	1    2450 6250
 	1    0    0    -1
 $EndComp
 $Comp
-L C C_BULK_5
+L C C_5VBULK_3
 U 1 1 57F9FD03
-P 4000 6250
-F 0 "C_BULK_5" H 4025 6350 50  0000 L CNN
-F 1 "10-100uF" H 4025 6150 50  0000 L CNN
-F 2 "Capacitors_SMD:C_1206_HandSoldering" H 4038 6100 50  0001 C CNN
-F 3 "" H 4000 6250 50  0000 C CNN
-	1    4000 6250
-	1    0    0    -1
-$EndComp
-$Comp
-L C C_BULK_6
-U 1 1 57F9FF08
-P 4500 6250
-F 0 "C_BULK_6" H 4525 6350 50  0000 L CNN
-F 1 "10-100uF" H 4525 6150 50  0000 L CNN
-F 2 "Capacitors_SMD:C_1206_HandSoldering" H 4538 6100 50  0001 C CNN
-F 3 "" H 4500 6250 50  0000 C CNN
-	1    4500 6250
-	1    0    0    -1
-$EndComp
-$Comp
-L C C_BULK_7
-U 1 1 57F9FF52
-P 5050 6250
-F 0 "C_BULK_7" H 5075 6350 50  0000 L CNN
-F 1 "10-100uF" H 5075 6150 50  0000 L CNN
-F 2 "Capacitors_SMD:C_1206_HandSoldering" H 5088 6100 50  0001 C CNN
-F 3 "" H 5050 6250 50  0000 C CNN
-	1    5050 6250
+P 3000 6250
+F 0 "C_5VBULK_3" H 3025 6350 50  0000 L CNN
+F 1 "10-100uF" H 3025 6150 50  0000 L CNN
+F 2 "Capacitors_SMD:C_1206_HandSoldering" H 3038 6100 50  0001 C CNN
+F 3 "" H 3000 6250 50  0000 C CNN
+	1    3000 6250
 	1    0    0    -1
 $EndComp
@@
 	1    0    0    -1
 $EndComp
-Wire Wire Line
-	1900 6100 5050 6100
-Connection ~ 3500 6100
-Connection ~ 3000 6100
+NoConn ~ 3500 2150
+NoConn ~ 3500 2300
+$Comp
+L CP C_5VBULK_1
+U 1 1 57FA3E62
+P 1900 6250
+F 0 "C_5VBULK_1" H 1925 6350 50  0000 L CNN
+F 1 "10-100uF" H 1925 6150 50  0000 L CNN
+F 2 "Capacitors_ThroughHole:C_Radial_D6.3_L11.2_P2.5" H 1938 6100 50  0001 C CNN
+F 3 "" H 1900 6250 50  0000 C CNN
+	1    1900 6250
+	1    0    0    -1
+$EndComp
 Connection ~ 2450 6100
-Wire Wire Line
-	1900 6400 5050 6400
 Connection ~ 2450 6400
-Connection ~ 3000 6400
-Connection ~ 3500 6400
-Connection ~ 4000 6100
-Connection ~ 4500 6100
-Connection ~ 4000 6400
-Connection ~ 4500 6400
 Wire Wire Line
 	3000 3650 4100 3650
@@
 Wire Wire Line
 	6300 1900 3500 1900
-NoConn ~ 3500 2150
-NoConn ~ 3500 2300
-$Comp
-L CP C_BULK_1
-U 1 1 57FA3E62
-P 1900 6250
-F 0 "C_BULK_1" H 1925 6350 50  0000 L CNN
-F 1 "10-100uF" H 1925 6150 50  0000 L CNN
-F 2 "Capacitors_ThroughHole:C_Radial_D6.3_L11.2_P2.5" H 1938 6100 50  0001 C CNN
-F 3 "" H 1900 6250 50  0000 C CNN
-	1    1900 6250
-	1    0    0    -1
-$EndComp
-$Comp
-L CP C_BULK_2
-U 1 1 57FA450D
-P 2450 6250
-F 0 "C_BULK_2" H 2475 6350 50  0000 L CNN
-F 1 "10-100uF" H 2475 6150 50  0000 L CNN
-F 2 "Capacitors_ThroughHole:C_Radial_D6.3_L11.2_P2.5" H 2488 6100 50  0001 C CNN
-F 3 "" H 2450 6250 50  0000 C CNN
-	1    2450 6250
-	1    0    0    -1
-$EndComp
-$Comp
-L CP C_BULK_3
-U 1 1 57FA45D2
-P 3000 6250
-F 0 "C_BULK_3" H 3025 6350 50  0000 L CNN
-F 1 "10-100uF" H 3025 6150 50  0000 L CNN
-F 2 "Capacitors_ThroughHole:C_Radial_D6.3_L11.2_P2.5" H 3038 6100 50  0001 C CNN
-F 3 "" H 3000 6250 50  0000 C CNN
-	1    3000 6250
-	1    0    0    -1
-$EndComp
 Wire Wire Line
 	1900 5800 1900 6100
 Wire Wire Line
 	1900 6400 1900 6750
+Wire Wire Line
+	1900 6400 3000 6400
+Wire Wire Line
+	1900 6100 3000 6100
 $EndSCHEMATC
