File: pcb/MainBoard/SectionCommBuffer.sch (KiCad schematic (older format))
At the start: 9 parts, among them U2 notgate_74HCT04

Commit message: PCB design finished
Parts:
- renumbered U2 to NOT1
Changed lines of the file:
@@
 $EndComp
 $Comp
-L GND #PWR021
+L GND #PWR019
 U 1 1 57FA05EC
 P 6850 4400
-F 0 "#PWR021" H 6850 4150 50  0001 C CNN
+F 0 "#PWR019" H 6850 4150 50  0001 C CNN
 F 1 "GND" H 6850 4250 50  0000 C CNN
 F 2 "" H 6850 4400 50  0000 C CNN
@@
 $EndComp
 $Comp
-L GND #PWR022
+L GND #PWR020
 U 1 1 57FA0B7B
 P 3200 2550
-F 0 "#PWR022" H 3200 2300 50  0001 C CNN
+F 0 "#PWR020" H 3200 2300 50  0001 C CNN
 F 1 "GND" H 3200 2400 50  0000 C CNN
 F 2 "" H 3200 2550 50  0000 C CNN
@@
 $EndComp
 $Comp
-L GND #PWR023
+L GND #PWR021
 U 1 1 57FA0C0F
 P 6850 1250
-F 0 "#PWR023" H 6850 1000 50  0001 C CNN
+F 0 "#PWR021" H 6850 1000 50  0001 C CNN
 F 1 "GND" H 6850 1100 50  0000 C CNN
 F 2 "" H 6850 1250 50  0000 C CNN
@@
 $EndComp
 $Comp
-L GND #PWR024
+L GND #PWR022
 U 1 1 57FA0CAD
 P 9750 1650
-F 0 "#PWR024" H 9750 1400 50  0001 C CNN
+F 0 "#PWR022" H 9750 1400 50  0001 C CNN
 F 1 "GND" H 9750 1500 50  0000 C CNN
 F 2 "" H 9750 1650 50  0000 C CNN
@@
 $EndComp
 $Comp
-L +5V #PWR025
+L +5V #PWR023
 U 1 1 57FA0D02
 P 2850 2250
-F 0 "#PWR025" H 2850 2100 50  0001 C CNN
+F 0 "#PWR023" H 2850 2100 50  0001 C CNN
 F 1 "+5V" H 2850 2390 50  0000 C CNN
 F 2 "" H 2850 2250 50  0000 C CNN
@@
 $EndComp
 $Comp
-L +5V #PWR026
+L +5V #PWR024
 U 1 1 57FA0D41
 P 6500 950
-F 0 "#PWR026" H 6500 800 50  0001 C CNN
+F 0 "#PWR024" H 6500 800 50  0001 C CNN
 F 1 "+5V" H 6500 1090 50  0000 C CNN
 F 2 "" H 6500 950 50  0000 C CNN
@@
 $EndComp
 $Comp
-L +5V #PWR027
+L +5V #PWR025
 U 1 1 57FA0D6C
 P 6500 4100
-F 0 "#PWR027" H 6500 3950 50  0001 C CNN
+F 0 "#PWR025" H 6500 3950 50  0001 C CNN
 F 1 "+5V" H 6500 4240 50  0000 C CNN
 F 2 "" H 6500 4100 50  0000 C CNN
@@
 $EndComp
 $Comp
-L +5V #PWR028
+L +5V #PWR026
 U 1 1 57FA0D8F
 P 9400 1350
-F 0 "#PWR028" H 9400 1200 50  0001 C CNN
+F 0 "#PWR026" H 9400 1200 50  0001 C CNN
 F 1 "+5V" H 9400 1490 50  0000 C CNN
 F 2 "" H 9400 1350 50  0000 C CNN
@@
 	1950 3650 2150 3650
 $Comp
-L +5V #PWR029
+L +5V #PWR027
 U 1 1 57FA10B1
 P 850 2950
-F 0 "#PWR029" H 850 2800 50  0001 C CNN
+F 0 "#PWR027" H 850 2800 50  0001 C CNN
 F 1 "+5V" H 850 3090 50  0000 C CNN
 F 2 "" H 850 2950 50  0000 C CNN
@@
 	850  3450 850  2950
 $Comp
-L GND #PWR030
+L GND #PWR028
 U 1 1 57FA10EA
 P 2150 3750
-F 0 "#PWR030" H 2150 3500 50  0001 C CNN
+F 0 "#PWR028" H 2150 3500 50  0001 C CNN
 F 1 "GND" H 2150 3600 50  0000 C CNN
 F 2 "" H 2150 3750 50  0000 C CNN
@@
 $EndComp
 $Comp
-L GND #PWR031
+L GND #PWR029
 U 1 1 57FA1156
 P 2600 4350
-F 0 "#PWR031" H 2600 4100 50  0001 C CNN
+F 0 "#PWR029" H 2600 4100 50  0001 C CNN
 F 1 "GND" H 2600 4200 50  0000 C CNN
 F 2 "" H 2600 4350 50  0000 C CNN
@@
 $EndComp
 $Comp
-L GND #PWR032
+L GND #PWR030
 U 1 1 57FA1262
 P 6300 3000
-F 0 "#PWR032" H 6300 2750 50  0001 C CNN
+F 0 "#PWR030" H 6300 2750 50  0001 C CNN
 F 1 "GND" H 6300 2850 50  0000 C CNN
 F 2 "" H 6300 3000 50  0000 C CNN
@@
 $EndComp
 $Comp
-L GND #PWR033
+L GND #PWR031
 U 1 1 57FA1286
 P 6300 6100
-F 0 "#PWR033" H 6300 5850 50  0001 C CNN
+F 0 "#PWR031" H 6300 5850 50  0001 C CNN
 F 1 "GND" H 6300 5950 50  0000 C CNN
 F 2 "" H 6300 6100 50  0000 C CNN
@@
 $EndComp
 $Comp
-L GND #PWR034
+L GND #PWR032
 U 1 1 57FA12AA
 P 9000 3400
-F 0 "#PWR034" H 9000 3150 50  0001 C CNN
+F 0 "#PWR032" H 9000 3150 50  0001 C CNN
 F 1 "GND" H 9000 3250 50  0000 C CNN
 F 2 "" H 9000 3400 50  0000 C CNN
@@
 FIFO_PUSH
 $Comp
-L notgate_74HCT04 U2
+L notgate_74HCT04 NOT1
 U 1 1 57FA151D
 P 4700 3550
-F 0 "U2" H 4850 3650 50  0000 C CNN
+F 0 "NOT1" H 4850 3650 50  0000 C CNN
 F 1 "notgate_74HCT04" H 5000 3400 50  0000 C CNN
 F 2 "Housings_SOIC:SOIC-14_3.9x8.7mm_Pitch1.27mm" H 4700 3550 50  0001 C CNN
@@
 	3550 3850 3700 3850
 $Comp
-L +5V #PWR035
+L +5V #PWR033
 U 1 1 57FA2552
 P 4650 3450
-F 0 "#PWR035" H 4650 3300 50  0001 C CNN
+F 0 "#PWR033" H 4650 3300 50  0001 C CNN
 F 1 "+5V" H 4650 3590 50  0000 C CNN
 F 2 "" H 4650 3450 50  0000 C CNN
@@
 $EndComp
 $Comp
-L GND #PWR036
+L GND #PWR034
 U 1 1 57FA25E4
 P 4650 3650
-F 0 "#PWR036" H 4650 3400 50  0001 C CNN
+F 0 "#PWR034" H 4650 3400 50  0001 C CNN
 F 1 "GND" H 4650 3500 50  0000 C CNN
 F 2 "" H 4650 3650 50  0000 C CNN
@@
 NoConn ~ 5700 2150
 $Comp
-L GND #PWR037
+L GND #PWR035
 U 1 1 57FA27F6
 P 5700 1800
-F 0 "#PWR037" H 5700 1550 50  0001 C CNN
+F 0 "#PWR035" H 5700 1550 50  0001 C CNN
 F 1 "GND" H 5700 1650 50  0000 C CNN
 F 2 "" H 5700 1800 50  0000 C CNN
@@
 $EndComp
 $Comp
-L GND #PWR038
+L GND #PWR036
 U 1 1 57FA281C
 P 5700 4900
-F 0 "#PWR038" H 5700 4650 50  0001 C CNN
+F 0 "#PWR036" H 5700 4650 50  0001 C CNN
 F 1 "GND" H 5700 4750 50  0000 C CNN
 F 2 "" H 5700 4900 50  0000 C CNN
@@
 $EndComp
 $Comp
-L GND #PWR039
+L GND #PWR037
 U 1 1 57FA28FF
 P 7100 1800
-F 0 "#PWR039" H 7100 1550 50  0001 C CNN
+F 0 "#PWR037" H 7100 1550 50  0001 C CNN
 F 1 "GND" H 7100 1650 50  0000 C CNN
 F 2 "" H 7100 1800 50  0000 C CNN
@@
 $EndComp
 $Comp
-L GND #PWR040
+L GND #PWR038
 U 1 1 57FA2925
 P 7100 4900
-F 0 "#PWR040" H 7100 4650 50  0001 C CNN
+F 0 "#PWR038" H 7100 4650 50  0001 C CNN
 F 1 "GND" H 7100 4750 50  0000 C CNN
 F 2 "" H 7100 4900 50  0000 C CNN
@@
 	7650 5200 10200 5200
 $Comp
-L GND #PWR041
+L GND #PWR039
 U 1 1 57FA3AFE
 P 8150 2000
-F 0 "#PWR041" H 8150 1750 50  0001 C CNN
+F 0 "#PWR039" H 8150 1750 50  0001 C CNN
 F 1 "GND" H 8150 1850 50  0000 C CNN
 F 2 "" H 8150 2000 50  0000 C CNN
