File: pcb/MainBoard/SectionMainControl.sch (KiCad schematic (older format))
At the start: 1 part, among them U3 arduino_mini

Commit message: PCB design finished
Parts:
- renumbered U3 to ARD2
Changed lines of the file:
@@
 $EndDescr
 $Comp
-L arduino_mini U3
+L arduino_mini ARD2
 U 1 1 57FA863B
 P 5000 3400
-F 0 "U3" H 5500 2450 70  0000 C CNN
+F 0 "ARD2" H 5550 2450 70  0000 C CNN
 F 1 "arduino_mini" H 5750 2350 70  0000 C CNN
 F 2 "arduino:arduino_mini" H 5000 3350 60  0001 C CNN
@@
 NoConn ~ 5150 2250
 $Comp
-L +5V #PWR042
+L +5V #PWR040
 U 1 1 57FA8701
 P 5000 2250
-F 0 "#PWR042" H 5000 2100 50  0001 C CNN
+F 0 "#PWR040" H 5000 2100 50  0001 C CNN
 F 1 "+5V" H 5000 2390 50  0000 C CNN
 F 2 "" H 5000 2250 50  0000 C CNN
@@
 $EndComp
 $Comp
-L GND #PWR043
+L GND #PWR041
 U 1 1 57FA8717
 P 5000 4950
-F 0 "#PWR043" H 5000 4700 50  0001 C CNN
+F 0 "#PWR041" H 5000 4700 50  0001 C CNN
 F 1 "GND" H 5000 4800 50  0000 C CNN
 F 2 "" H 5000 4950 50  0000 C CNN

Commit message: re-assigned data ready from pin 10 to pin 7.
Connections:
- net FIFO_DATA_READY: now also ARD2.25 (D7); no longer ARD2.28 ((SS)#D10)
Changed lines of the file:
@@
 Wire Wire Line
 	5700 2850 6500 2850
-Text HLabel 6500 3050 2    60   Input ~ 0
+Text HLabel 6500 3350 2    60   Input ~ 0
 FIFO_DATA_READY
 Text HLabel 6500 3250 2    60   Output ~ 0
@@
 Text HLabel 6500 3150 2    60   Output ~ 0
 FIFO_ENABLE
-Wire Wire Line
-	5700 3050 6500 3050
 Wire Wire Line
 	5700 3150 6500 3150
@@
 NoConn ~ 5700 4000
 NoConn ~ 5700 3800
-NoConn ~ 5700 3350
 NoConn ~ 5700 2950
+Wire Wire Line
+	5700 3350 6500 3350
+NoConn ~ 5700 3050
 $EndSCHEMATC
